File: hc-sippy-cad/hc-sippy.sch (EAGLE design)
At the start: 11 parts

Commit message: schematic update
Parts:
- R1, R2: value 1K -> 1.5K
Changed lines of the file:
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@@
 <part name="SW_RST" library="adafruit" deviceset="SWITCH_PUSHBUTTON" device="EVQ-PE"/>
 <part name="SUPPLY1" library="supply2" library_urn="urn:adsk.eagle:library:372" deviceset="GND" device=""/>
-<part name="R1" library="akstudios-adafruit" deviceset="R-US_" device="0309/12" value="1K"/>
-<part name="R2" library="akstudios-adafruit" deviceset="R-US_" device="0309/12" value="1K"/>
+<part name="R1" library="akstudios-adafruit" deviceset="R-US_" device="0309/12" value="1.5K"/>
+<part name="R2" library="akstudios-adafruit" deviceset="R-US_" device="0309/12" value="1.5K"/>
 <part name="LED_RST" library="akstudios-adafruit" deviceset="LED" device="5MM"/>
 <part name="LED_SIP" library="akstudios-adafruit" deviceset="LED" device="5MM"/>
